File: corne-cherry/pcb/corne-cherry.kicad_pcb (KiCad board)
At the start: 2 copper layers, 275.5 x 105.6 mm, 172 parts, among them J1 MJ-4PP-9, J2 OLED, J3 MJ-4PP-9, J4 OLED, SW1 SW_PUSH, SW10 SW_PUSH, SW11 SW_PUSH, SW12 SW_PUSH, SW13 SW_PUSH, SW14 SW_PUSH, SW15 SW_PUSH, SW16 SW_PUSH, SW17 SW_PUSH, SW18 SW_PUSH, SW19 SW_PUSH, SW2 SW_PUSH, SW20 SW_PUSH, SW21 SW_PUSH, SW22 SW_PUSH, SW23 SW_PUSH, SW24 SW_PUSH, SW25 SW_PUSH, SW26 SW_PUSH, SW27 SW_PUSH, SW28 SW_PUSH, SW29 SW_PUSH, SW3 SW_PUSH, SW30 SW_PUSH, SW31 SW_PUSH, SW32 SW_PUSH, SW33 SW_PUSH, SW34 SW_PUSH, SW35 SW_PUSH, SW36 SW_PUSH, SW37 SW_PUSH, SW38 SW_PUSH, SW39 SW_PUSH, SW4 SW_PUSH, SW40 SW_PUSH, SW41 SW_PUSH, SW42 SW_PUSH, SW5 SW_PUSH, SW6 SW_PUSH, SW7 SW_PUSH, SW8 SW_PUSH, SW9 SW_PUSH, U1 ProMicro, U2 ProMicro

Commit message: corne-cherry.kicad_sch: changed the components in the circuit diagram to make the corne fit the seeed xiao ble.
Parts:
- added D1: LED_PERM, LED_SMD:LED_0603_1608Metric, F.Cu at (104.0, 126.9)
- added D22: LED_PERM, LED_SMD:LED_0603_1608Metric, F.Cu at (104.0, 129.4)
- added D43: LED_PERM, LED_SMD:LED_0603_1608Metric, F.Cu at (15.1, 127.1)
- added D44: LED_PERM, LED_SMD:LED_0603_1608Metric, F.Cu at (15.1, 129.7)
- added D45: LED_PERM, LED_SMD:LED_0603_1608Metric, F.Cu at (15.1, 132.2)
- added D46: LED_PERM, LED_SMD:LED_0603_1608Metric, F.Cu at (15.1, 134.7)
- added D47: LED_PERM, LED_SMD:LED_0603_1608Metric, F.Cu at (15.1, 137.3)
- added D48: LED_PERM, LED_SMD:LED_0603_1608Metric, F.Cu at (104.0, 132.0)
- added D49: LED_PERM, LED_SMD:LED_0603_1608Metric, F.Cu at (104.0, 134.5)
- added D50: LED_PERM, LED_SMD:LED_0603_1608Metric, F.Cu at (104.0, 137.1)
- added J1: CONN_DISPLAY_SOCKET, Connector_PinSocket_1.27mm:PinSocket_1x05_P1.27mm_Vertical, F.Cu at (17.6, 147.4)
- added J2: Conn_01x02, Connector_AMASS:AMASS_XT30PW-F_1x02_P2.50mm_Horizontal, F.Cu at (50.6, 158.7)
- added J4: CONN_DISPLAY_SOCKET, Connector_PinSocket_1.27mm:PinSocket_1x05_P1.27mm_Vertical, F.Cu at (112.4, 147.2)
- added J5: Conn_01x02, Connector_AMASS:AMASS_XT30PW-F_1x02_P2.50mm_Horizontal, F.Cu at (148.9, 161.2)
- added R1: R_LED_PERM, Resistor_SMD:R_0603_1608Metric, F.Cu at (20.1, 127.1)
- added R10: R_LED_PERM, Resistor_SMD:R_0603_1608Metric, F.Cu at (110.7, 137.1)
- added R2: R_LED_PERM, Resistor_SMD:R_0603_1608Metric, F.Cu at (20.9, 129.7)
- added R3: R_LED_PERM, Resistor_SMD:R_0603_1608Metric, F.Cu at (20.1, 132.2)
- added R4: R_LED_PERM, Resistor_SMD:R_0603_1608Metric, F.Cu at (20.1, 134.7)
- added R5: R_LED_PERM, Resistor_SMD:R_0603_1608Metric, F.Cu at (20.9, 137.3)
- added R6: R_LED_PERM, Resistor_SMD:R_0603_1608Metric, F.Cu at (110.7, 126.9)
- added R7: R_LED_PERM, Resistor_SMD:R_0603_1608Metric, F.Cu at (110.7, 129.4)
- added R8: R_LED_PERM, Resistor_SMD:R_0603_1608Metric, F.Cu at (110.7, 132.0)
- added R9: R_LED_PERM, Resistor_SMD:R_0603_1608Metric, F.Cu at (110.7, 134.5)
- added SW43: SW_RGB_UNDERGLOW, Button_Switch_SMD:SW_SPDT_CK-JS102011SAQN, F.Cu at (34.7, 129.8)
- added SW44: SW_RGB_PERKEY, Button_Switch_SMD:SW_SPDT_CK-JS102011SAQN, F.Cu at (34.7, 139.6)
- added SW45: SW_RGB_LED_OLED, Button_Switch_SMD:SW_SPDT_CK-JS102011SAQN, F.Cu at (34.7, 149.4)
- added SW46: SW_RGB_PERKEY, Button_Switch_SMD:SW_SPDT_CK-JS102011SAQN, F.Cu at (34.7, 159.2)
- added SW47: SW_RGB_PERKEY, Button_Switch_SMD:SW_SPDT_CK-JS102011SAQN, F.Cu at (127.6, 157.6)
- added SW48: SW_RGB_LED_OLED, Button_Switch_SMD:SW_SPDT_CK-JS102011SAQN, F.Cu at (126.7, 127.6)
- added SW49: SW_RGB_UNDERGLOW, Button_Switch_SMD:SW_SPDT_CK-JS102011SAQN, F.Cu at (126.7, 137.4)
- added SW50: SW_RGB_PERKEY, Button_Switch_SMD:SW_SPDT_CK-JS102011SAQN, F.Cu at (126.7, 147.2)
- added U1: xiao-ble, Seeed Studio XIAO Series Library:XIAO-nRF52840-Sense-14P-2.54-21X17.8MM, F.Cu at (57.2, 132.5)
- added U2: xiao-ble, Seeed Studio XIAO Series Library:XIAO-nRF52840-Sense-14P-2.54-21X17.8MM, F.Cu at (147.6, 133.0)
Connections:
- D13 pad 1: row2 -> row3
- D28 pad 1: row1_r -> row3_r
- D34 pad 1: row2_r -> row3_r
- D7 pad 1: row1 -> row3
- LED1 pad 1: VCC -> VCC_LED_UNDERGLOW
- LED10 pad 1: VCC -> VCC_LED_PERKEY
- LED11 pad 1: VCC -> VCC_LED_PERKEY
- LED12 pad 1: VCC -> VCC_LED_PERKEY
- LED13 pad 1: VCC -> VCC_LED_PERKEY
- LED13 pad 2: Net-(LED13-Pad2) -> unconnected-(LED13-DOUT-Pad2)
- LED14 pad 1: VCC -> VCC_LED_PERKEY
- LED15 pad 1: VCC -> VCC_LED_PERKEY
- LED16 pad 1: VCC -> VCC_LED_PERKEY
- LED17 pad 1: VCC -> VCC_LED_PERKEY
- LED18 pad 1: VCC -> VCC_LED_PERKEY
- LED2 pad 1: VCC -> VCC_LED_UNDERGLOW
- LED20 pad 1: VCC -> VCC_LED_PERKEY
- LED21 pad 1: VCC -> VCC_LED_PERKEY
- LED22 pad 1: VCC -> VCC_LED_PERKEY
- LED23 pad 1: VCC -> VCC_LED_PERKEY
- LED24 pad 1: VCC -> VCC_LED_PERKEY
- LED25 pad 1: VCC -> VCC_LED_PERKEY
- LED26 pad 1: VCC -> VCC_LED_PERKEY
- LED27 pad 1: VCC -> VCC_LED_PERKEY
- LED28 pad 1: VDD -> VCC_LED_R_UNDERGLOW
- LED28 pad 2: Net-(LED28-Pad2) -> Net-(LED28-DOUT)
- LED29 pad 1: VDD -> VCC_LED_R_UNDERGLOW
- LED3 pad 1: VCC -> VCC_LED_UNDERGLOW
- LED30 pad 1: VDD -> VCC_LED_R_UNDERGLOW
- LED31 pad 1: VDD -> VCC_LED_R_UNDERGLOW
- LED31 pad 2: Net-(LED31-Pad2) -> Net-(LED28-DOUT)
- LED31 pad 4: Net-(LED28-Pad2) -> Net-(LED28-DOUT)
- LED32 pad 1: VDD -> VCC_LED_R_UNDERGLOW
- LED32 pad 2: Net-(LED32-Pad2) -> Net-(LED28-DOUT)
- LED32 pad 4: Net-(LED31-Pad2) -> Net-(LED28-DOUT)
- LED33 pad 1: VDD -> VCC_LED_R_UNDERGLOW
- LED33 pad 2: Net-(LED33-Pad2) -> Net-(LED28-DOUT)
- LED33 pad 4: Net-(LED32-Pad2) -> Net-(LED28-DOUT)
- LED34 pad 1: VDD -> VCC_LED_R_PERKEY
- LED35 pad 1: VDD -> VCC_LED_R_PERKEY
- LED36 pad 1: VDD -> VCC_LED_R_PERKEY
- LED37 pad 1: VDD -> VCC_LED_R_PERKEY
- LED38 pad 1: VDD -> VCC_LED_R_PERKEY
- LED39 pad 1: VDD -> VCC_LED_R_PERKEY
- LED4 pad 1: VCC -> VCC_LED_UNDERGLOW
- LED40 pad 1: VDD -> VCC_LED_R_PERKEY
- LED40 pad 2: Net-(LED40-Pad2) -> unconnected-(LED40-DOUT-Pad2)
- LED41 pad 1: VDD -> VCC_LED_R_PERKEY
- LED42 pad 1: VDD -> VCC_LED_R_PERKEY
- LED43 pad 1: VDD -> VCC_LED_R_PERKEY
- LED44 pad 1: VDD -> VCC_LED_R_PERKEY
- LED45 pad 1: VDD -> VCC_LED_R_PERKEY
- LED47 pad 1: VDD -> VCC_LED_R_PERKEY
- LED48 pad 1: VDD -> VCC_LED_R_PERKEY
- LED49 pad 1: VDD -> VCC_LED_R_PERKEY
- LED5 pad 1: VCC -> VCC_LED_UNDERGLOW
- LED50 pad 1: VDD -> VCC_LED_R_PERKEY
- LED51 pad 1: VDD -> VCC_LED_R_PERKEY
- LED52 pad 1: VDD -> VCC_LED_R_PERKEY
- LED53 pad 1: VDD -> VCC_LED_R_PERKEY
- LED54 pad 1: VDD -> VCC_LED_R_PERKEY
- LED54 pad 4: Net-(LED33-Pad2) -> Net-(LED28-DOUT)
- LED6 pad 1: VCC -> VCC_LED_UNDERGLOW
- LED7 pad 1: VCC -> VCC_LED_PERKEY
- LED8 pad 1: VCC -> VCC_LED_PERKEY
- LED9 pad 1: VCC -> VCC_LED_PERKEY
- SW13 pad 1: col0 -> col2
- SW28 pad 1: col0_r -> col1_r
- SW34 pad 1: col0_r -> col2_r
- SW7 pad 1: col0 -> col1
Routing:
- net Net-(LED28-DOUT): track 0.00 -> 193.6 mm, vias 0 -> 6
- net Net-(LED31-Pad2): track 71.8 -> 0.00 mm, vias 2 -> 0
- net Net-(LED32-Pad2): track 47.4 -> 0.00 mm
- net Net-(LED28-Pad2): track 41.5 -> 0.00 mm, vias 2 -> 0
- net Net-(LED33-Pad2): track 32.9 -> 0.00 mm, vias 2 -> 0
- net col2_r: vias 5 -> 10
- net col2: vias 5 -> 10
- net col0_r: vias 5 -> 0
- net col0: vias 5 -> 0
Other:
- board size 275.5 x 105.6 mm -> 295.5 x 105.6 mm
