File: corne-cherry/pcb/corne-cherry.kicad_sch (KiCad schematic)
At the start: 146 parts, among them J1 MJ-4PP-9, J2 OLED, J3 MJ-4PP-9, J4 OLED, SW1 SW_PUSH, SW10 SW_PUSH, SW11 SW_PUSH, SW12 SW_PUSH, SW13 SW_PUSH, SW14 SW_PUSH, SW15 SW_PUSH, SW16 SW_PUSH, SW17 SW_PUSH, SW18 SW_PUSH, SW19 SW_PUSH, SW2 SW_PUSH, SW20 SW_PUSH, SW21 SW_PUSH, SW22 SW_PUSH, SW23 SW_PUSH, SW24 SW_PUSH, SW25 SW_PUSH, SW26 SW_PUSH, SW27 SW_PUSH, SW28 SW_PUSH, SW29 SW_PUSH, SW3 SW_PUSH, SW30 SW_PUSH, SW31 SW_PUSH, SW32 SW_PUSH, SW33 SW_PUSH, SW34 SW_PUSH, SW35 SW_PUSH, SW36 SW_PUSH, SW37 SW_PUSH, SW38 SW_PUSH, SW39 SW_PUSH, SW4 SW_PUSH, SW40 SW_PUSH, SW41 SW_PUSH, SW42 SW_PUSH, SW5 SW_PUSH, SW6 SW_PUSH, SW7 SW_PUSH, SW8 SW_PUSH, SW9 SW_PUSH, U1 ProMicro, U2 ProMicro

Commit message: corne-cherry.kicad_sch: changed the components in the circuit diagram to make the corne fit the seeed xiao ble.
Parts:
- removed D1, D22: D, kbd:D3_SMD_v2, symbol Device:D
- removed J1, J3: MJ-4PP-9, kbd:MJ-4PP-9_1side, symbol kbd:MJ-4PP-9
- removed J2, J4: OLED, kbd:OLED_1side, symbol Connector_Generic:Conn_01x04
- removed LED19, LED46: YS-SK6812MINI-E, kbd:YS-SK6812MINI-E, symbol kbd:YS-SK6812MINI-E
- removed SW1, SW22: SW_PUSH, kbd:CherryMX_Hotswap, symbol kbd:SW_PUSH
- removed U1, U2: ProMicro, kbd:ProMicro_v3, symbol kbd:ProMicro
- added D1, D22, D43, D44, D45, D46, D47, D48, D49, D50: LED_PERM, LED_SMD:LED_0603_1608Metric, symbol Device:LED
- added J1, J4: CONN_DISPLAY_SOCKET, Connector_PinSocket_1.27mm:PinSocket_1x05_P1.27mm_Vertical, symbol Connector:Conn_01x05_Socket
- added J2, J5: Conn_01x02, Connector_AMASS:AMASS_XT30PW-F_1x02_P2.50mm_Horizontal, symbol Connector_Generic:Conn_01x02
- added R1, R10, R2, R3, R4, R5, R6, R7, R8, R9: R_LED_PERM, Resistor_SMD:R_0603_1608Metric, symbol Device:R_Small
- added SW43, SW49: SW_RGB_UNDERGLOW, Button_Switch_SMD:SW_SPDT_CK-JS102011SAQN, symbol Switch:SW_Push_SPDT
- added SW44, SW46, SW47, SW50: SW_RGB_PERKEY, Button_Switch_SMD:SW_SPDT_CK-JS102011SAQN, symbol Switch:SW_Push_SPDT
- added SW45, SW48: SW_RGB_LED_OLED, Button_Switch_SMD:SW_SPDT_CK-JS102011SAQN, symbol Switch:SW_Push_SPDT
- added U1, U2: xiao-ble, Seeed Studio XIAO Series Library:XIAO-nRF52840-Sense-14P-2.54-21X17.8MM, symbol keyboard_mcu:xiao-ble
Connections:
- net GND: now also D43.1 (K), D44.1 (K), D45.1 (K), D46.1 (K), D47.1 (K), J1.4 (Pin_4), U1.13 (GND)
- net GNDA: now also D1.1 (K), D22.1 (K), D48.1 (K), D49.1 (K), D50.1 (K), J4.4 (Pin_4), U2.13 (GND)
- net LED: now also SW45.3 (C)
- net LED_r: now also SW48.3 (C)
- net SCL: now also J1.2 (Pin_2), U1.6 (A9_SCL/0.05_H)
- net SCL_r: now also J4.2 (Pin_2), U2.6 (A9_SCL/0.05_H)
- net SDA: now also J1.1 (Pin_1), SW45.1 (A)
- net SDA_r: now also J4.1 (Pin_1), SW48.1 (A)
- net VCC: now also J1.3 (Pin_3), J1.5 (Pin_5), SW43.2 (B), SW44.2 (B), SW46.2 (B), U1.12 (3V3); no longer LED1.1 (VDD), LED10.1 (VDD), LED11.1 (VDD), LED12.1 (VDD), LED13.1 (VDD), LED14.1 (VDD), LED15.1 (VDD), LED16.1 (VDD), LED17.1 (VDD), LED18.1 (VDD), LED2.1 (VDD), LED20.1 (VDD), LED21.1 (VDD), LED22.1 (VDD), LED23.1 (VDD), LED24.1 (VDD), LED25.1 (VDD), LED26.1 (VDD), LED27.1 (VDD), LED3.1 (VDD), LED4.1 (VDD), LED5.1 (VDD), LED6.1 (VDD), LED7.1 (VDD), LED8.1 (VDD), LED9.1 (VDD)
- net VDD: now also J4.3 (Pin_3), J4.5 (Pin_5), SW47.2 (B), SW49.2 (B), SW50.2 (B), U2.12 (3V3); no longer LED28.1 (VDD), LED29.1 (VDD), LED30.1 (VDD), LED31.1 (VDD), LED32.1 (VDD), LED33.1 (VDD), LED34.1 (VDD), LED35.1 (VDD), LED36.1 (VDD), LED37.1 (VDD), LED38.1 (VDD), LED39.1 (VDD), LED40.1 (VDD), LED41.1 (VDD), LED42.1 (VDD), LED43.1 (VDD), LED44.1 (VDD), LED45.1 (VDD), LED47.1 (VDD), LED48.1 (VDD), LED49.1 (VDD), LED50.1 (VDD), LED51.1 (VDD), LED52.1 (VDD), LED53.1 (VDD), LED54.1 (VDD)
- net col1: now also SW7.1, U1.7 (B8_TX/1.11)
- net col1_r: now also SW28.1, U2.7 (B8_TX/1.11)
- net col2: now also SW13.1, U1.11 (A6_MOSI/1.15)
- net col2_r: now also SW34.1, U2.11 (A6_MOSI/1.15)
- net col3: now also U1.10 (A5_MISO/1.14)
- net col3_r: now also U2.10 (A5_MISO/1.14)
- net col4: now also U1.9 (A7_SCK/1.13)
- net col4_r: now also U2.9 (A7_SCK/1.13)
- net col5: now also U1.8 (B9_RX/1.12)
- net col5_r: now also U2.8 (B9_RX/1.12)
- net reset: now also U1.17 (RESET)
- net reset_r: now also U2.17 (RESET)
- net row0: now also U1.1 (A2/0.02_H)
- net row0_r: now also U2.1 (A2/0.02_H)
- net row1: now also U1.2 (A4/0.03_H); no longer D7.1 (K)
- net row1_r: now also U2.2 (A4/0.03_H); no longer D28.1 (K)
- net row2: now also U1.3 (A10/0.28); no longer D13.1 (K)
- net row2_r: now also U2.3 (A10/0.28); no longer D34.1 (K)
- net row3: now also D13.1 (K), D7.1 (K), U1.4 (A11/0.29)
- net row3_r: now also D28.1 (K), D34.1 (K), U2.4 (A11/0.29)
- net at LED33.2 (DOUT), LED54.4 (DIN): now also LED28.2 (DOUT), LED31.2 (DOUT), LED31.4 (DIN), LED32.2 (DOUT), LED32.4 (DIN), LED33.4 (DIN)
- removed net col0: SW13.1, SW7.1
- removed net col0_r: SW28.1, SW34.1
- new net: D43.2 (A), R1.1
- new net: D22.2 (A), R7.1
- new net: J2.1 (Pin_1), U1.20 (GND)
- new net: J2.2 (Pin_2), U1.19 (BAT)
- new net: D49.2 (A), R9.1
- new net: J5.1 (Pin_1), U2.20 (GND)
- new net: J5.2 (Pin_2), U2.19 (BAT)
- new net: D45.2 (A), R3.1
- new net: D50.2 (A), R10.1
- new net: D1.2 (A), R6.1
- new net: D48.2 (A), R8.1
- new net: D44.2 (A), R2.1
- new net: D46.2 (A), R4.1
- new net: D47.2 (A), R5.1
- new net SDA_LED: SW45.2 (B), U1.5 (A8_SDA/0.04_H)
- new net SDA_R_LED: SW48.2 (B), U2.5 (A8_SDA/0.04_H)
- new net VCC_LED_PERKEY: LED10.1 (VDD), LED11.1 (VDD), LED12.1 (VDD), LED13.1 (VDD), LED14.1 (VDD), LED15.1 (VDD), LED16.1 (VDD), LED17.1 (VDD), LED18.1 (VDD), LED20.1 (VDD), LED21.1 (VDD), LED22.1 (VDD), LED23.1 (VDD), LED24.1 (VDD), LED25.1 (VDD), LED26.1 (VDD), LED27.1 (VDD), LED7.1 (VDD), LED8.1 (VDD), LED9.1 (VDD), SW44.3 (C)
- new net VCC_LED_PERM: R1.2, R2.2, R3.2, R4.2, R5.2, SW46.3 (C)
- new net VCC_LED_R_PERKEY: LED34.1 (VDD), LED35.1 (VDD), LED36.1 (VDD), LED37.1 (VDD), LED38.1 (VDD), LED39.1 (VDD), LED40.1 (VDD), LED41.1 (VDD), LED42.1 (VDD), LED43.1 (VDD), LED44.1 (VDD), LED45.1 (VDD), LED47.1 (VDD), LED48.1 (VDD), LED49.1 (VDD), LED50.1 (VDD), LED51.1 (VDD), LED52.1 (VDD), LED53.1 (VDD), LED54.1 (VDD), SW50.3 (C)
- new net VCC_LED_R_PERM: R10.2, R6.2, R7.2, R8.2, R9.2, SW47.3 (C)
- new net VCC_LED_R_UNDERGLOW: LED28.1 (VDD), LED29.1 (VDD), LED30.1 (VDD), LED31.1 (VDD), LED32.1 (VDD), LED33.1 (VDD), SW49.3 (C)
- new net VCC_LED_UNDERGLOW: LED1.1 (VDD), LED2.1 (VDD), LED3.1 (VDD), LED4.1 (VDD), LED5.1 (VDD), LED6.1 (VDD), SW43.3 (C)
- no-connect marks 14 -> 20
Other:
- moved on the sheet: D10, D11, D12, D13, D14, D15, D16, D17, D18, D19, D2, D20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

Commit message: finished track routing.
Parts:
- removed J5: Conn_01x02, Connector_AMASS:AMASS_XT30PW-F_1x02_P2.50mm_Horizontal, symbol Connector_Generic:Conn_01x02
- removed RSW1, RSW2: SW_PUSH, kbd:ResetSW_1side, symbol kbd:SW_PUSH
- removed SW43, SW49: SW_RGB_UNDERGLOW, Button_Switch_SMD:SW_SPDT_CK-JS102011SAQN, symbol Switch:SW_Push_SPDT
- removed SW44, SW50: SW_RGB_PERKEY, Button_Switch_SMD:SW_SPDT_CK-JS102011SAQN, symbol Switch:SW_Push_SPDT
- removed SW45, SW48: SW_RGB_LED_OLED, Button_Switch_SMD:SW_SPDT_CK-JS102011SAQN, symbol Switch:SW_Push_SPDT
- added J3: Conn_01x02, Connector_JST:JST_PH_S2B-PH-K_1x02_P2.00mm_Horizontal, symbol Connector_Generic:Conn_01x02
- added J5, J6, J7, J8: Conn_01x01_Socket, Jumper:SolderJumper-2_P1.3mm_Bridged_RoundedPad1.0x1.5mm, symbol Connector:Conn_01x01_Socket
- added JP1, JP2: SolderJumper, Jumper:SolderJumper-3_P1.3mm_Open_Pad1.0x1.5mm_NumberLabels, symbol Jumper:SolderJumper_3_Open
- added SW1: SW_ONOFF, Button_Switch_SMD:SW_SPDT_PCM12, symbol Switch:SW_Push_SPDT
- added SW22: SW_ONOFF_R, Button_Switch_SMD:SW_SPDT_PCM12, symbol Switch:SW_Push_SPDT
- D7: footprint kbd:D3_SMD_v2 -> foolstan_kbd:D3_SMD_v2
- J1, J4: footprint Connector_PinSocket_1.27mm:PinSocket_1x05_P1.27mm_Vertical -> Connector_PinSocket_2.54mm:PinSocket_1x05_P2.54mm_Vertical
- J2: footprint Connector_AMASS:AMASS_XT30PW-F_1x02_P2.50mm_Horizontal -> Connector_JST:JST_PH_S2B-PH-K_1x02_P2.00mm_Horizontal
- SW46, SW47: value SW_RGB_PERKEY -> SW_LED_PERM; footprint Button_Switch_SMD:SW_SPDT_CK-JS102011SAQN -> Button_Switch_SMD:SW_SPDT_PCM12
- U1, U2: footprint Seeed Studio XIAO Series Library:XIAO-nRF52840-Sense-14P-2.54-21X17.8MM -> Seeed Studio XIAO Series Library:XIAO-Generic-Thruhole-14P-2.54-21X17.8MM
Connections:
- net VCC_LED_PERKEY is gone; now on net VCC: LED10.1 (VDD), LED11.1 (VDD), LED12.1 (VDD), LED13.1 (VDD), LED14.1 (VDD), LED15.1 (VDD), LED16.1 (VDD), LED17.1 (VDD), LED18.1 (VDD), LED20.1 (VDD), LED21.1 (VDD), LED22.1 (VDD), LED23.1 (VDD), LED24.1 (VDD), LED25.1 (VDD), LED26.1 (VDD), LED27.1 (VDD), LED7.1 (VDD), LED8.1 (VDD), LED9.1 (VDD)
- net VCC_LED_R_PERKEY is gone; now on net VDD: LED34.1 (VDD), LED35.1 (VDD), LED36.1 (VDD), LED37.1 (VDD), LED38.1 (VDD), LED39.1 (VDD), LED40.1 (VDD), LED41.1 (VDD), LED42.1 (VDD), LED43.1 (VDD), LED44.1 (VDD), LED45.1 (VDD), LED47.1 (VDD), LED48.1 (VDD), LED49.1 (VDD), LED50.1 (VDD), LED51.1 (VDD), LED52.1 (VDD), LED53.1 (VDD), LED54.1 (VDD)
- net VCC_LED_R_UNDERGLOW is gone; now on net VDD: LED28.1 (VDD), LED29.1 (VDD), LED30.1 (VDD), LED31.1 (VDD), LED32.1 (VDD), LED33.1 (VDD)
- net VCC_LED_UNDERGLOW is gone; now on net VCC: LED1.1 (VDD), LED2.1 (VDD), LED3.1 (VDD), LED4.1 (VDD), LED5.1 (VDD), LED6.1 (VDD)
- net LED: now also JP1.3 (B)
- net LED_r: now also JP2.3 (B)
- net SDA: now also JP1.1 (A)
- net SDA_LED: now also JP1.2 (C)
- net SDA_R_LED: now also JP2.2 (C)
- net SDA_r: now also JP2.1 (A)
- net VCC_LED_PERM: now also SW46.1 (A); no longer SW46.3 (C)
- net VCC_LED_R_PERM: now also SW47.1 (A); no longer SW47.3 (C)
- net at J2.1 (Pin_1): now also SW1.3 (C); no longer U1.20 (GND)
- net at J2.2 (Pin_2): now also J5.1 (Pin_1); no longer U1.19 (BAT)
- net reset: no longer names the net of U1.17 (RESET)
- net reset_r: no longer names the net of U2.17 (RESET)
- new net: LED33.2 (DOUT), LED54.4 (DIN)
- new net: LED28.2 (DOUT), LED31.4 (DIN)
- new net: LED32.2 (DOUT), LED33.4 (DIN)
- new net: LED31.2 (DOUT), LED32.4 (DIN)
- new net: J3.1 (Pin_1), SW22.3 (C)
- new net: J3.2 (Pin_2), J6.1 (Pin_1)
- new net: J7.1 (Pin_1), SW1.2 (B)
- new net: J8.1 (Pin_1), SW22.2 (B)
- no-connect marks 20 -> 24
Other:
- title: Corne Cherry -> Corne Cherry Panda
- moved on the sheet: J1, J2, J4, SW46, SW47
